File: vesuvius-badge/vesuvius-badge.kicad_pcb (KiCad board)
At the start: 2 copper layers, 137.5 x 86 mm, 65 parts, among them U1 MAX7219

Commit message: some routing done
Routing:
- net Net-(D10-Pad1): track 0.00 -> 264.5 mm, vias 0 -> 12
- net Net-(D13-Pad1): track 0.00 -> 240.0 mm, vias 0 -> 8
- net Net-(D14-Pad1): track 0.00 -> 239.7 mm, vias 0 -> 16
- net Net-(D33-Pad2): track 0.00 -> 233.8 mm, vias 0 -> 12
- net Net-(D25-Pad2): track 0.00 -> 225.9 mm, vias 0 -> 21
- net Net-(D41-Pad2): track 0.00 -> 225.7 mm, vias 0 -> 10
- net Net-(D17-Pad2): track 0.00 -> 215.2 mm, vias 0 -> 14
- net Net-(D16-Pad1): track 0.00 -> 207.1 mm, vias 0 -> 14
- net Net-(D12-Pad1): track 0.00 -> 206.0 mm, vias 0 -> 23
- net Net-(D15-Pad1): track 0.00 -> 192.4 mm, vias 0 -> 14
- net Net-(D49-Pad2): track 0.00 -> 191.3 mm, vias 0 -> 18
- net Net-(D11-Pad1): track 0.00 -> 188.9 mm, vias 0 -> 16
- net Net-(D1-Pad1): track 0.00 -> 188.2 mm, vias 0 -> 23
- net Net-(D1-Pad2): track 0.00 -> 185.6 mm, vias 0 -> 14
- net Net-(D57-Pad2): track 0.00 -> 174.8 mm, vias 0 -> 16
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