File: vesuvius-badge/vesuvius-badge-charlie/vesuvius-badge-charlie.kicad_pcb (KiCad board)
At the start: 2 copper layers, 162.5 x 85.5 mm, 166 parts, among them J1 Conn_01x05, J2 Conn_01x03, U1 IS31FL3731-QF, U2 Pico, U3 CH32V003J4M6

Commit message: latest changes
Other:
- board text removed: "JLCJLCJLCJLC"
Changed lines of the file:
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@@
     (effects (font (size 1 1) (thickness 0.15)) (justify mirror))
-  )
-  (gr_text "JLCJLCJLCJLC" (at 247.25 88.75) (layer "B.SilkS")
-    (effects (font (size 1.5 1.5) (thickness 0.3)) (justify mirror))
   )
   (gr_text "INTB" (at 223.75 65.25 45) (layer "B.SilkS")
